Commit message: Update crazyflie 2 model

File: rotors_description/urdf/crazyflie2.xacro (robot description, xacro)
@@ -1,3 +1,4 @@
 <?xml version="1.0"?>
+<!-- Created by Lakshman Kumar ( lkumar93@terpmailumd.edu ) -->
 <robot name="crazyflie2" xmlns:xacro="http://ros.org/wiki/xacro">
   <!-- Properties -->
@@ -9,8 +10,8 @@
   <xacro:property name="body_width" value="0.092" /> <!--av [m] -->
   <xacro:property name="body_height" value="0.029" /> <!--av [m] -->
-  <xacro:property name="mass_rotor" value="0.0027" /> <!-- av [kg] -->
+  <xacro:property name="mass_rotor" value="0.0003" /> <!-- av [kg] -->
   <xacro:property name="arm_length" value="0.02275" /> <!--  0.03973 av [m] -->
   <xacro:property name="rotor_offset_top" value="0.013" /> <!-- av [m] -->
-  <xacro:property name="radius_rotor" value="0.023" /> <!-- av [m] -->
+  <xacro:property name="radius_rotor" value="0.02275" /> <!-- av [m] -->
   <xacro:property name="motor_constant" value="8.54858e-06" /> <!-- [kg.m/s^2] -->
   <xacro:property name="moment_constant" value="0.005" /> <!-- av [m] -->
@@ -27,7 +28,7 @@
     <inertia ixx="2.3951e-5" ixy="0.0" ixz="0.0" iyy="2.3951e-5" iyz="0.0" izz="3.2347e-5" /> <!-- [kg.m^2] [kg.m^2] [kg.m^2] [kg.m^2] [kg.m^2] [kg.m^2] -->
   </xacro:property>
-  <!-- inertia of a single rotor, assuming it is a cuboid. Height=3mm, width=15mm -->
+  <!-- inertia of a single rotor, assuming it is a cuboid. Height=0.7mm, width=0.3mm -->
   <xacro:property name="rotor_inertia">
-    <xacro:box_inertia x="${radius_rotor}" y="0.016" z="0.003" mass="${mass_rotor*rotor_velocity_slowdown_sim}" />
+    <xacro:box_inertia x="${radius_rotor}" y="0.007" z="0.003" mass="${mass_rotor*rotor_velocity_slowdown_sim}" />
   </xacro:property>
   <!-- Included URDF Files -->

File: rotors_description/urdf/crazyflie2_base.xacro (robot description, xacro)
@@ -1,3 +1,4 @@
 <?xml version="1.0"?>
+<!-- Created by Lakshman Kumar ( lkumar93@terpmail.umd.edu ) -->
 <robot name="crazyflie2" xmlns:xacro="http://ros.org/wiki/xacro">
   <xacro:include filename="$(find rotors_description)/urdf/component_snippets.xacro" />
@@ -16,5 +17,5 @@
       parent_link="${namespace}/base_link"
       imu_topic="imu"
-      mass_imu_sensor="0.002"
+      mass_imu_sensor="0.001"
       gyroscope_noise_density="0.0003394"
       gyroscopoe_random_walk="0.000038785"
